Commit message: Add files via upload

File: diffbot_description/urdf/diffbot.urdf.xacro (robot description, xacro)
@@ -5,4 +5,11 @@
   <link name="left_wheel_link"/>
   <link name="right_wheel_link"/>
+  <link name="imu_link"/>
+  <joint name="imu_joint" type="fixed">
+    <parent link="base_link"/>
+    <child link="imu_link"/>
+    <!-- IMU가 base_link 기준 어디에 붙었는지. 모르면 일단 0 -->
+    <origin xyz="0 0 0" rpy="0 0 0"/>
+  </joint>
   <!-- ========== Joints (중요: joint 이름이 ros2_control과 일치해야 함) ========== -->
   <joint name="left_wheel_joint" type="continuous">
@@ -24,9 +31,11 @@
     <hardware>
       <plugin>opencr_diffbot_hw/OpenCRSystem</plugin>
-      <!-- OpenCR 쪽 시리얼 포트/속도: Step 4~5에서 info_.hardware_parameters로 읽음 -->
+      <!-- OpenCR serial parameters -->
       <param name="device">/dev/ttyACM0</param>
       <param name="baud">115200</param>
     </hardware>
-    <!-- 조인트 2개: 이 이름이 OpenCRSystem::on_init()에서 읽는 info_.joints[0], [1]로 들어옴 -->
+    <!-- ========================= -->
+    <!-- Actuated joints (wheels)  -->
+    <!-- ========================= -->
     <joint name="left_wheel_joint">
       <command_interface name="velocity"/>
@@ -39,4 +48,22 @@
       <state_interface name="velocity"/>
     </joint>
+    <!-- ========================= -->
+    <!-- IMU sensor declaration   -->
+    <!-- ========================= -->
+    <sensor name="imu">
+      <!-- Orientation (quaternion) -->
+      <state_interface name="orientation.x"/>
+      <state_interface name="orientation.y"/>
+      <state_interface name="orientation.z"/>
+      <state_interface name="orientation.w"/>
+      <!-- Angular velocity (rad/s) -->
+      <state_interface name="angular_velocity.x"/>
+      <state_interface name="angular_velocity.y"/>
+      <state_interface name="angular_velocity.z"/>
+      <!-- Linear acceleration (m/s^2) -->
+      <state_interface name="linear_acceleration.x"/>
+      <state_interface name="linear_acceleration.y"/>
+      <state_interface name="linear_acceleration.z"/>
+    </sensor>
   </ros2_control>
 </robot>
